File: aio3-tut/aio3-tut.kicad_pcb (KiCad board)
At the start: 2 copper layers, 24 parts, among them J1 USB_B, SW1 SW_Push, U1 ATmega32U4-AU, Y1 16MHz

Commit message: placed
Parts:
- C3, C4, C5, C6, C7, F1, J1, R1, R2, R3, R4, SW1: moved to B.Cu
- moved SW1 152.0 mm to (85.8, 133.6), turned to 270 degrees
- moved C4 147.7 mm to (101.7, 132.1), turned to 90 degrees
- moved C7 130.3 mm to (109.1, 131.8), turned to 270 degrees
- moved C6 124.8 mm to (119.1, 118.3), turned to 90 degrees
- moved C3 113.6 mm to (94.5, 120.1), turned to 270 degrees
- moved R1 107.7 mm to (84.1, 121.4), turned to 90 degrees
- moved R2 104.7 mm to (90.5, 113.7), turned to 90 degrees
- moved R4 98.0 mm to (116.7, 129.4), turned to 270 degrees
- moved J1 96.4 mm to (84.4, 98.0), turned to 270 degrees
- moved F1 94.2 mm to (82.5, 109.2), turned to 90 degrees
- moved C5 64.8 mm to (119.9, 107.4), turned to 90 degrees
- moved R3 49.5 mm to (95.0, 113.5), turned to 90 degrees
- moved C2 14.3 mm to (102.4, 106.4)
- moved MX1 13.3 mm to (145.1, 108.0)
- moved D1 13.3 mm to (153.0, 108.7)
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